File: KiCad_MiniBadge_Learning.kicad_pcb (KiCad board)
At the start: 2 copper layers, 20.4 x 20.3 mm, 10 parts, among them U1 SAINTCON-Simple

Commit message: Add files via upload
Parts:
- D2: moved to B.Cu
Other:
- board text added: "I learned KiCad minibadge creating with RuShan"
