File: KiCad_MiniBadge_Learning.kicad_sch (KiCad schematic)
At the start: 7 parts, among them U1 SAINTCON-Simple

Commit message: Add files via upload
Parts:
- R1: value RESISTOR1206 -> 68 ohm
Other:
- moved on the sheet: D1, D2, JP1, JP2, R1, R2, U1
